File: PCBs/v1.0/Main PCB/KiCAD/MRF-Pro-v7.5.kicad_pcb (KiCad board)
At the start: 2 copper layers, 56.5 x 28.7 mm, 6 parts, among them J1 Feather-1, J2 Feather-2, J3 FPC 8P Connector, J4 Conn_01x08

Commit message: fix(pcb): put v7.5 FPC pin 1 on the switched rail instead of D11
FPC pin 1 ran to Feather D11, left over from a PWM experiment that was
never pursued. The breakout ties FPC pins 1 and 6 to the same 3.3 V net,
so the strap did nothing but reserve a GPIO and hang an unused pin on the
supply.

Pin 1 now joins pin 6 on 3V3_SW, the rail the J4 switch gates, so both
boards agree and the supply crosses the ribbon on two conductors instead
of one. D11 is free again. Boards already built are unaffected: they were
always powered through pin 6, and the firmware never drives D11.

ERC and DRC match the previous board exactly (same single wire-endpoint
warning, same 11 warnings, no unconnected pads). Zones refilled, Gerbers
and drill files re-plotted. Saving from KiCad 10 also upgrades the board
and project file format.

Docs and the v1 harness diagrams follow the change, and three stale J4
pin 7/8 references in the v8 errata now match the board.
Connections:
- J2 pad 7: Net-(J2-Pin_7) -> unconnected-(J2-Pin_7-Pad7)
- J3 pad 1: Net-(J2-Pin_7) -> /3V3_SW
- J3 pad 6: Net-(J3-Pin_6) -> /3V3_SW
- J4 pad 8: Net-(J3-Pin_6) -> /3V3_SW
Routing:
- net Net-(J2-Pin_7): track 35.2 -> 0.00 mm, vias 2 -> 0
- net /3V3_SW: track 0.00 -> 24.6 mm
- net Net-(J3-Pin_6): track 14.8 -> 0.00 mm
