File: PCBs/v2.0/Main PCB/KiCAD/MRF-Pro-v8.kicad_pcb (KiCad board)
At the start: 2 copper layers, 56.5 x 28.7 mm, 6 parts, among them J1 Feather-1, J2 Feather-2, J3 FPC 8P Connector, J4 Conn_01x08

Commit message: fix(pcb): make v2 main board J4 a right-angle socket
The main board's connectors are meant to be right angle, matching the
breakout. J4 was the odd one out: a top-entry land, which is what forced
the top-entry part number in the previous commit. Swap the footprint to
JST_SH_SM08B-SRSS-TB_1x08-1MP_P1.00mm_Horizontal so the harness leaves
over the board edge, and put C7430450 (ZX-SH1.0-8PWT) back on the BOM.

The pad row moves 2.83mm east to x=160.4978, so the connector is nudged
0.5mm inboard to keep the courtyard off the edge - it now clears by
0.31mm, with 0.86mm from the outer pads to the edge. Pad Y positions are
unchanged and six of the eight stubs just extend east.

Two nets needed real work. 3.3OUT's via at (159.675, 105.5) ended up
overlapping pad 7, a different net, so it moves to (159.675, 107.6) with
a 45-degree stub down from pad 8. Net-(J2-Pin_6) lost its escape route
entirely - it used to reach the old pad from the east, through the strip
the new pads now occupy - and is rerouted on the back layer, passing
north of the EN via rather than squeezing past it.

Zones refilled, DRC clean (0 errors, 0 unconnected; the three remaining
warnings are pre-existing library mismatches on J1/J2/J3). Gerbers and
drill re-plotted; only the ten J4 pads move, every other layer differs by
timestamp alone. J4's CPL row follows the pad bounding box centre, as the
rest of the file does.

v1 is deliberately untouched and stays top entry, so the README and the
wiring table now split J4 by revision.
Parts:
- J4: footprint Connector_JST:JST_SH_BM08B-SRSS-TB_1x08-1MP_P1.00mm_Vertical -> JST_SH_SM08B-SRSS-TB_1x08-1MP_P1.00mm_Horizontal
- moved J4 0.50 mm to (158.5, 102.6)
Routing:
- net Net-(J2-Pin_6): track 38.8 -> 28.9 mm, vias 0 -> 2
- net GND: track 11.0 -> 19.5 mm
- net Net-(J2-Pin_5): track 27.4 -> 30.2 mm
- net EN: track 39.3 -> 42.1 mm
- net 3.3IN: track 75.5 -> 78.3 mm
- net 3.3OUT: track 12.7 -> 10.2 mm
