File: PCBs/v2.0/Main PCB/KiCAD/MRF-Pro-v8.kicad_sch (KiCad schematic)
At the start: 6 parts, among them J1 Feather-1, J2 Feather-2, J3 FPC 8P Connector, J4 Conn_01x08

Commit message: fix(pcb): use the top-entry SH1.0 part for main board J4
J4's footprint is JST_SH_BM08B-SRSS-TB_1x08-1MP_P1.00mm_Vertical, a
top-entry land: signal pads at local y=+1.325, mounting pegs at y=-1.2,
2.525mm apart. The BOM called out C7430450, which is a Megastar
ZX-SH1.0-8PWT - the WT suffix means right angle. Its JST equivalent,
SM08B-SRSS-TB, wants 3.875mm between the signal row and the pegs, so the
leads sit about 1.35mm off a 1.55mm pad. JLCPCB's DFM check caught it on
a builder's order.

The wrong number came from the breakout, where the WT family is right:
J6 and J7 sit on SM04B/SM06B Horizontal footprints. J4 was the only one
paired against a Vertical footprint. It also carried a 6-pin number
before 3020700, so JLC used to reject it on pin count and nobody got as
far as the land pattern.

C7430457 is the same connector in the LT (top entry) variant. Footprint,
gerbers and CPL are unchanged - it is a part swap only, on both board
revisions.

Also names the entry direction in the README parts list so the LT/WT
suffix is not a trap for the next person ordering.
Parts:
- J4: LCSC C7430450 -> C7430457
Changed lines of the file:
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@@
 			)
 		)
-		(property "LCSC" "C7430450"
+		(property "LCSC" "C7430457"
 			(at 104.14 49.53 90)
 			(hide yes)

Commit message: fix(pcb): make v2 main board J4 a right-angle socket
The main board's connectors are meant to be right angle, matching the
breakout. J4 was the odd one out: a top-entry land, which is what forced
the top-entry part number in the previous commit. Swap the footprint to
JST_SH_SM08B-SRSS-TB_1x08-1MP_P1.00mm_Horizontal so the harness leaves
over the board edge, and put C7430450 (ZX-SH1.0-8PWT) back on the BOM.

The pad row moves 2.83mm east to x=160.4978, so the connector is nudged
0.5mm inboard to keep the courtyard off the edge - it now clears by
0.31mm, with 0.86mm from the outer pads to the edge. Pad Y positions are
unchanged and six of the eight stubs just extend east.

Two nets needed real work. 3.3OUT's via at (159.675, 105.5) ended up
overlapping pad 7, a different net, so it moves to (159.675, 107.6) with
a 45-degree stub down from pad 8. Net-(J2-Pin_6) lost its escape route
entirely - it used to reach the old pad from the east, through the strip
the new pads now occupy - and is rerouted on the back layer, passing
north of the EN via rather than squeezing past it.

Zones refilled, DRC clean (0 errors, 0 unconnected; the three remaining
warnings are pre-existing library mismatches on J1/J2/J3). Gerbers and
drill re-plotted; only the ten J4 pads move, every other layer differs by
timestamp alone. J4's CPL row follows the pad bounding box centre, as the
rest of the file does.

v1 is deliberately untouched and stays top entry, so the README and the
wiring table now split J4 by revision.
Parts:
- J4: footprint Connector_JST:JST_SH_BM08B-SRSS-TB_1x08-1MP_P1.00mm_Vertical -> Connector_JST:JST_SH_SM08B-SRSS-TB_1x08-1MP_P1.00mm_Horizontal; LCSC C7430457 -> C7430450
Changed lines of the file:
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@@
 			)
 		)
-		(property "Footprint" "Connector_JST:JST_SH_BM08B-SRSS-TB_1x08-1MP_P1.00mm_Vertical"
+		(property "Footprint" "Connector_JST:JST_SH_SM08B-SRSS-TB_1x08-1MP_P1.00mm_Horizontal"
 			(at 104.14 49.53 0)
 			(hide yes)
@@
 			)
 		)
-		(property "LCSC" "C7430457"
+		(property "LCSC" "C7430450"
 			(at 104.14 49.53 90)
 			(hide yes)
